File: KiCAD/ZCU111_DAC/FEA.kicad_pcb (KiCad board)
At the start: 4 copper layers, 73.1 x 34 mm, 53 parts, among them U1 SMA, U11 SMA, U12 SMA, U13 TCM2-33WX+, U14 SMA, U15 SMA, U16 TCM2-33WX+, U2 SMA, U3 SMA, U4 LMH6702MF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

Commit message: update
Parts:
- removed C6: 0.1uF, Capacitors_SMD:C_0603
- removed U9: SMA, MyFootprints:SMA_side_mount
- added C11: 0.1uF, Capacitors_SMD:C_0603, B.Cu at (47.0, 170.8)
- added C12: 0.1uF, Capacitors_SMD:C_0603, B.Cu at (47.0, 172.2)
- added C13: 0.1uF, Capacitors_SMD:C_0603, B.Cu at (56.5, 170.8)
- added C14: 0.1uF, Capacitors_SMD:C_0603, B.Cu at (56.5, 172.4)
- added P1: CONN_01X04, Pin_Headers:Pin_Header_Straight_1x04_Pitch2.54mm, F.Cu at (22.2, 159.6)
- moved U8 12.5 mm to (86.1, 158.7), turned to 90 degrees
- moved C5 6.80 mm to (85.2, 163.0), turned to 0 degrees
- moved U14 2.84 mm to (28.2, 161.7)
- moved U15 2.19 mm to (27.7, 171.2)
- moved U1 1.42 mm to (36.5, 161.7)
- moved U2 0.91 mm to (36.0, 171.2)
- moved C7 0.22 mm to (53.5, 171.1)
- moved C10 0.13 mm to (43.9, 171.0)
Connections:
- C10 pad 2: VCC12_SW -> 5V
- C7 pad 2: VCC12_SW -> 5V
- C8 pad 2: VCC12_SW -> 5V
- C9 pad 2: VCC12_SW -> 5V
- U4 pad 2: Earth -> -5V
- U4 pad 6: VCC12_SW -> 5V
- U6 pad 2: Earth -> -5V
- U6 pad 6: VCC12_SW -> 5V
- U7 pad A35: VCC1V8_BUS -> (no net)
- U7 pad C35: VCC1V8_BUS -> (no net)
Routing:
- net Earth: track 12.2 -> 61.1 mm, vias 2 -> 4
- net -5V: track 0.00 -> 8.67 mm, vias 0 -> 2
- net UTIL_3V3: track 42.1 -> 50.4 mm
- net 5V: track 0.00 -> 5.68 mm, vias 0 -> 1
- net RFMC_DAC_00_P: track 18.2 -> 14.6 mm
- net RFMC_DAC_00_N: track 26.7 -> 23.7 mm
- net VCC12_SW: track 6.95 -> 5.08 mm
- net RFMC_DAC_01_N: track 27.0 -> 25.5 mm
- added copper zone on F.Cu, net -5V
- added copper zone on In2.Cu, net 5V
- removed copper zone on F.Cu, net UTIL_3V3
- removed copper zone on In2.Cu, net VCC12_SW
Other:
- board text added: "GND VEE GNE VCC"
- board text removed: "VCC12"
