File: KiCAD/ZCU111_DAC/FEA.sch (KiCad schematic (older format))
At the start: 53 parts, among them U1 SMA, U11 SMA, U12 SMA, U13 TCM2-33WX+, U14 SMA, U15 SMA, U16 TCM2-33WX+, U2 SMA, U3 SMA, U4 LMH6702MF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

Commit message: update
Parts:
- removed C6: 0.1uF, Capacitors_SMD:C_0603, symbol device:C
- removed U9: SMA, MyFootprints:SMA_side_mount, symbol Mylibrary:SMA
- added C11, C12, C13, C14: 0.1uF, Capacitors_SMD:C_0603, symbol device:C
- added P1: CONN_01X04, Pin_Headers:Pin_Header_Straight_1x04_Pitch2.54mm, symbol conn:CONN_01X04
Connections:
- net Earth: now also C11.1, C12.1, C13.1, C14.1, P1.2 (P2), P1.4 (P4); no longer U4.2 (V-), U6.2 (V-)
- net VCC12_SW: no longer C10.2, C7.2, C8.2, C9.2, U4.6 (V+), U6.6 (V+)
- net VCC1V8_BUS: no longer names the net of U7.A35 (35)
- net VCC1V8_BUS: no longer U7.C35 (35)
- new net -5V: C11.2, C12.2, C13.2, C14.2, P1.3 (P3), U4.2 (V-), U6.2 (V-)
- new net 5V: C10.2, C7.2, C8.2, C9.2, P1.1 (P1), U4.6 (V+), U6.6 (V+)
- no-connect marks 53 -> 55
Other:
- moved on the sheet: C10, C7, C8, C9, R10, R11, R12, R13, R14, R15, R16, R17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
